File: rev1.a/LIR2032Charger.kicad_pcb (KiCad board)
At the start: 2 copper layers, 36.8 x 26.8 mm, 12 parts, among them J1 USB_A_PLUG, U1 MCP73831

Commit message: fixed erc errors and added gerber files
Routing:
- net Net-(BT1-Pad1): track 12.2 -> 45.8 mm
- net /+5V: track 32.0 -> 51.1 mm
- net Net-(LED1-Pad1): track 0.05 -> 7.46 mm
Changed lines of the file:
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@@
   (general
     (links 20)
-    (no_connects 3)
-    (area 104.024999 81.914656 141.005344 108.885344)
+    (no_connects 0)
+    (area 102.32 79.57 143.310001 111.510001)
     (thickness 1.6)
     (drawings 14)
-    (tracks 58)
+    (tracks 76)
     (zones 0)
     (modules 12)
@@
     (visible_elements 7FFEFFFF)
     (pcbplotparams
-      (layerselection 0x00030_ffffffff)
-      (usegerberextensions false)
+      (layerselection 0x010f0_ffffffff)
+      (usegerberextensions true)
       (excludeedgelayer true)
       (linewidth 0.100000)
@@
       (plotinvisibletext false)
       (padsonsilk false)
-      (subtractmaskfromsilk false)
+      (subtractmaskfromsilk true)
       (outputformat 1)
       (mirror false)
-      (drillshape 1)
+      (drillshape 0)
       (scaleselection 1)
-      (outputdirectory ""))
+      (outputdirectory Gerber/))
   )
   (net 0 "")
@@
   (segment (start 135.04902 90.5) (end 136.34 90.5) (width 0.254) (layer F.Cu) (net 1))
   (via (at 136.34 90.5) (size 0.8) (drill 0.4) (layers F.Cu B.Cu) (net 1))
+  (segment (start 128.48 91.65) (end 128.48 86.875) (width 0.508) (layer F.Cu) (net 2))
+  (segment (start 128.48 86.875) (end 126.45 84.845) (width 0.508) (layer F.Cu) (net 2))
+  (segment (start 129.44 92.61) (end 128.48 91.65) (width 0.508) (layer F.Cu) (net 2))
+  (segment (start 130.25 92.61) (end 129.44 92.61) (width 0.508) (layer F.Cu) (net 2))
+  (segment (start 136.87 99.23) (end 130.25 92.61) (width 0.508) (layer F.Cu) (net 2))
+  (segment (start 136.87 101.31) (end 136.87 99.23) (width 0.508) (layer F.Cu) (net 2))
+  (segment (start 132.225 105.955) (end 136.87 101.31) (width 0.508) (layer F.Cu) (net 2))
+  (segment (start 126.45 105.955) (end 132.225 105.955) (width 0.508) (layer F.Cu) (net 2))
   (segment (start 126 94) (end 126 85.295) (width 0.508) (layer F.Cu) (net 2))
   (segment (start 126 85.295) (end 126.45 84.845) (width 0.508) (layer F.Cu) (net 2))
@@
   (segment (start 124.6 94) (end 126 94) (width 0.508) (layer F.Cu) (net 2))
   (segment (start 123.38 94.53) (end 124.07 94.53) (width 0.508) (layer F.Cu) (net 2))
+  (segment (start 131.89 102.47) (end 132.95098 101.40902) (width 0.508) (layer F.Cu) (net 3))
+  (segment (start 132.95098 101.40902) (end 132.95098 100.3) (width 0.508) (layer F.Cu) (net 3))
+  (segment (start 121.27 102.47) (end 131.89 102.47) (width 0.508) (layer F.Cu) (net 3))
+  (segment (start 118 99.2) (end 121.27 102.47) (width 0.508) (layer F.Cu) (net 3))
+  (segment (start 118 98) (end 118 99.2) (width 0.508) (layer F.Cu) (net 3))
   (segment (start 118.8 92.4) (end 119.45 91.75) (width 0.508) (layer F.Cu) (net 3))
   (segment (start 119.45 91.75) (end 119.45 90.5) (width 0.508) (layer F.Cu) (net 3))
@@
   (segment (start 109 99.21) (end 116.79 99.21) (width 0.508) (layer F.Cu) (net 3))
   (segment (start 118 96.5) (end 117.5 96.5) (width 0.25) (layer F.Cu) (net 3))
+  (segment (start 134.6 98.83) (end 135.04902 99.27902) (width 0.254) (layer F.Cu) (net 6))
+  (segment (start 135.04902 99.27902) (end 135.04902 100.3) (width 0.254) (layer F.Cu) (net 6))
+  (segment (start 131.72 98.83) (end 134.6 98.83) (width 0.254) (layer F.Cu) (net 6))
+  (segment (start 130.25 100.3) (end 131.72 98.83) (width 0.254) (layer F.Cu) (net 6))
+  (segment (start 129.45 100.3) (end 130.25 100.3) (width 0.254) (layer F.Cu) (net 6))
   (segment (start 129.45 100) (end 129.5 100) (width 0.25) (layer F.Cu) (net 6))
   (segment (start 132.95098 90.5) (end 129.45 90.5) (width 0.254) (layer F.Cu) (net 7))
